File: Coco_pico_keyb.kicad_sch (KiCad schematic)
At the start: 10 parts, among them J1 Conn_01x16_Pin, J2 DE9_Plug_MountingHoles, J3 Conn_01x16_Pin, U1 Pico

Commit message: Update board layout
Parts:
- removed JP2: OPEN=HOST, Jumper:SolderJumper-2_P1.3mm_Open_RoundedPad1.0x1.5mm, symbol Jumper:SolderJumper_2_Bridged
- added D3: Schottky (e.g. SS14), symbol Device:D
- added D4, D5, D6, D7, D8: BAT54S, Package_TO_SOT_SMD:SOT-23, symbol Diode:BAT54S
- added J4: SSD1306 I2C Display (optional), Connector_PinHeader_2.54mm:PinHeader_1x04_P2.54mm_Vertical, symbol Connector_Generic:Conn_01x04
- added J5: Power In, Connector_PinHeader_2.54mm:PinHeader_1x02_P2.54mm_Vertical, symbol Connector_Generic:Conn_01x02
- added J6: Remote DE9, Connector_PinHeader_2.54mm:PinHeader_2x05_P2.54mm_Vertical, symbol Connector_Generic:Conn_02x05_Odd_Even
- added SW1: Pairing Button, Button_Switch_THT:SW_PUSH_6mm, symbol Switch:SW_Push
Connections:
- net GND: now reaches D1.2 (A), D2.2 (A), JP1.2 (B), U1.23 (GND)
- net GND: now also D4.1 (A), D5.1 (A), D6.1 (A), D7.1 (A), D8.1 (A), J4.2 (Pin_2), J5.2 (Pin_2), J6.8 (Pin_8), SW1.2
- net GPIO27_ADC1: now reaches J2.1, U1.32 (GPIO27_ADC1)
- net GPIO27_ADC1: now also D4.3 (COM), J6.1 (Pin_1)
- net GPIO20: now reaches J2.2, U1.26 (GPIO20)
- net GPIO20: now also D5.3 (COM), J6.2 (Pin_2)
- net GPIO21: now reaches J2.3, U1.27 (GPIO21)
- net GPIO21: now also D6.3 (COM), J6.3 (Pin_3)
- net GPIO22: now reaches J2.4, U1.29 (GPIO22)
- net GPIO22: now also D7.3 (COM), J6.4 (Pin_4)
- net at J2.5: now also U1.40 (VBUS)
- net GPIO26_ADC0: now reaches J2.6, U1.31 (GPIO26_ADC0)
- net GPIO26_ADC0: now also D8.3 (COM), J6.6 (Pin_6)
- net I2C0_SDA: now reaches U1.21 (GPIO16)
- net I2C0_SDA: now also J4.4 (Pin_4)
- net DRAGON_SEL: now reaches JP1.1 (A)
- net DRAGON_SEL: now also U1.34 (GPIO28_ADC2); no longer U1.22 (GPIO17)
- net BTN_PAIR: now reaches U1.10 (GPIO7)
- net BTN_PAIR: now also SW1.1
- net 3V3: now reaches U1.36 (3V3)
- net 3V3: now also D4.2 (K), D5.2 (K), D6.2 (K), D7.2 (K), D8.2 (K), J4.1 (Pin_1)
- net VSYS: now reaches U1.39 (VSYS)
- net VSYS: now also D3.1 (K)
- new net I2C0_SCL: J4.3 (Pin_3), U1.22 (GPIO17)
- new net J5_VIN: D3.2 (A), J5.1 (Pin_1)
