File: _autosave-Coco_pico_keyb.kicad_pcb (KiCad board)
At the start: 2 copper layers, 65.5 x 70.5 mm, 13 parts, among them J1 Conn_01x16_Pin, J2 DE9_Plug_MountingHoles, J3 Conn_01x16_Pin, U1 Pico

Commit message: updates
Parts:
- renumbered REF** to mnt1, REF** to mnt2, REF** to mnt3
Changed lines of the file:
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@@
 		(descr "Mounting Hole 3.2mm, no annular, M3")
 		(tags "mounting hole 3.2mm no annular m3")
-		(property "Reference" "REF**"
+		(property "Reference" "mnt1"
 			(at 0 -4.2 0)
 			(layer "F.SilkS")
@@
 		(descr "Mounting Hole 3.2mm, no annular, M3")
 		(tags "mounting hole 3.2mm no annular m3")
-		(property "Reference" "REF**"
+		(property "Reference" "mnt3"
 			(at 0 -4.2 0)
 			(layer "F.SilkS")
@@
 		(descr "Mounting Hole 3.2mm, no annular, M3")
 		(tags "mounting hole 3.2mm no annular m3")
-		(property "Reference" "REF**"
+		(property "Reference" "mnt2"
 			(at 0 -4.2 0)
 			(layer "F.SilkS")
